Commit message: Update kinect.urdf.xacro

File: drone/sensors/kinect.urdf.xacro (robot description, xacro)
@@ -24,5 +24,5 @@
        <origin xyz=" 0 0 0 " rpy="0 0 0" />
        <geometry>
-         <mesh filename="package://autonomous_drone/models/kinect.dae"/>
+         <mesh filename="package://drone/models/kinect.dae"/>
        </geometry>
      </visual>
