Commit message: Update sonar_sensor.urdf.xacro

File: drone/sensors/sonar_sensor.urdf.xacro (robot description, xacro)
@@ -19,5 +19,5 @@
         <geometry>
           <!--<box size="0.01 0.01 0.01" /> -->
-          <mesh filename="package://autonomous_drone/models/max_sonar_ez4.dae"/>
+          <mesh filename="package://drone/models/max_sonar_ez4.dae"/>
         </geometry>
       </visual>
