Commit message: Update bodyNsensors.urdf.xacro

File: drone/plugins/bodyNsensors.urdf.xacro (robot description, xacro)
@@ -6,6 +6,6 @@
 <xacro:property name="M_PI" value="3.1415926535897931" />
     <!-- Included gazebo simulation plugins and controller -->
-  <xacro:include filename="$(find autonomous_drone)/plugins/gazebo_sim_plugins.urdf.xacro" />
-  <xacro:include filename="$(find autonomous_drone)/plugins/gazebo_sim_controller.urdf.xacro" />
+  <xacro:include filename="$(find drone)/plugins/gazebo_sim_plugins.urdf.xacro" />
+  <xacro:include filename="$(find drone)/plugins/gazebo_sim_controller.urdf.xacro" />
   <!-- Combining Gazebo Plugins as gazebo_quadrotor_plugins -->
   <xacro:macro name="gazebo_quadrotor_plugins">
@@ -25,5 +25,5 @@
         <origin xyz="0 0 0" rpy="0 0 0" />
         <geometry>
-          <mesh filename="package://autonomous_drone/models/quadrotor_3.dae"/>
+          <mesh filename="package://drone/models/quadrotor_3.dae"/>
         </geometry>
       </visual>
@@ -31,5 +31,5 @@
         <origin xyz="0 0 0" rpy="0 0 0" />
         <geometry>
-          <mesh filename="package://autonomous_drone/models/quadrotor_4.stl"/>
+          <mesh filename="package://drone/models/quadrotor_4.stl"/>
         </geometry>
       </collision>
@@ -43,10 +43,10 @@
 <!-- //////////////////////// Seperated from main body and generic quadrotor plugins  //////////////////////////-->
     <!-- Hokuyo Laser sensor gazebo plugin  -->
-    <xacro:include filename="$(find autonomous_drone)/sensors/hokuyo_utm30lx.urdf.xacro" />
+    <xacro:include filename="$(find drone)/sensors/hokuyo_utm30lx.urdf.xacro" />
       <xacro:hokuyo_utm30lx name="laser" parent="base_link" ros_topic="scan" update_rate="40" ray_count="1081" min_angle="135" max_angle="-135">
       <origin xyz="0.0 0.0 0.08" rpy="3.14 0 0"/>
     </xacro:hokuyo_utm30lx>
     <!-- Hokuyo Laser sensor gazebo plugin  -->
-    <xacro:include filename="$(find autonomous_drone)/sensors/sonar_sensor.urdf.xacro" />
+    <xacro:include filename="$(find drone)/sensors/sonar_sensor.urdf.xacro" />
       <xacro:sonar_sensor name="sonar" parent="base_link" ros_topic="sonar_height" update_rate="10" min_range="0.01" max_range="3.0" field_of_view="${40*M_PI/180}" ray_count="3">
       <origin xyz="-0.15 0.0 0.0" rpy="0 ${90*M_PI/180} 0"/>

Commit message: Update bodyNsensors.urdf.xacro

File: drone/plugins/bodyNsensors.urdf.xacro (robot description, xacro)
@@ -25,5 +25,5 @@
         <origin xyz="0 0 0" rpy="0 0 0" />
         <geometry>
-          <mesh filename="package://drone/models/quadrotor_3.dae"/>
+          <mesh filename="package://drone/models/quadrotor_4.dae"/>
         </geometry>
       </visual>

Commit message: Update bodyNsensors.urdf.xacro

File: drone/plugins/bodyNsensors.urdf.xacro (robot description, xacro)
@@ -53,7 +53,7 @@
     </xacro:sonar_sensor>
     <!-- Kinect sensor gazebo plugin  -->
-   <!--<xacro:include filename="$(find drone)/sensors/kinect.urdf.xacro" />
-      <xacro:kinect parent_frame="base_link">
-      <origin xyz="0.0 0.0 0.18" rpy="0 0 0"/>
-    </xacro:kinect>-->
+    <xacro:include filename="$(find drone)/sensors/generic_camera.urdf.xacro" />
+    <xacro:generic_camera name="front" sim_name="ardrone" parent="base_link" update_rate="60" res_x="640" res_y="360" image_format="R8G8B8" hfov="${81*M_PI/180}">
+      <origin xyz="0.21 0.0 0.07" rpy="0 0 0"/>
+    </xacro:generic_camera
 </robot>
